Commit message: commit

File: install/llm_ros2/share/llm_ros2/urdf/bbot.ros2_control.xacro (robot description, xacro)
@@ -74,6 +74,6 @@
             <grip_count_threshold>4</grip_count_threshold>
             <max_grip_count>8</max_grip_count>
-            <release_tolerance>0.01</release_tolerance>
-            <disable_collisions_on_attach>false</disable_collisions_on_attach>
+            <release_tolerance>0.012</release_tolerance>
+            <disable_collisions_on_attach>true</disable_collisions_on_attach>
             <contact_topic>__default_topic__</contact_topic>
             </plugin>

File: install/llm_ros2/share/llm_ros2/urdf/mbot_arm_gazebo.xacro (robot description, xacro)
@@ -33,5 +33,5 @@
     <xacro:property name="right_gripper_height" value="0.01" />
     <xacro:property name="sqirt_3" value="1.732"/>
-    <xacro:property name="gripper_width" value="0.03"/>
+    <xacro:property name="gripper_width" value="0.05"/>
     <xacro:property name="gripper_len" value="0.005"/>
     <xacro:property name="gripper_hight"   value="0.01"/>
@@ -172,5 +172,5 @@
             <origin xyz="0.25 0 0.15" rpy="0 0 0" />
             <axis xyz="0 0 1" />
-            <limit effort="30" velocity="1" lower="-2.96" upper="2.96"/>
+            <limit effort="1" velocity="1" lower="-2.96" upper="2.96"/>
             <dynamics damping="50" friction="1"/>
         </joint>
@@ -198,5 +198,5 @@
             <origin xyz="0 0 ${link1_len}" rpy="0 0 0" />
             <axis xyz="1 0 0" />
-            <limit effort="30" velocity="1" lower="-2.35" upper="2.35" />
+            <limit effort="1" velocity="1" lower="-2.35" upper="2.35" />
             <dynamics damping="50" friction="1"/>
         </joint>
@@ -224,5 +224,5 @@
             <origin xyz="0 0 ${link2_len}" rpy="0 0 0" />
             <axis xyz="1 0 0" />
-            <limit effort="30" velocity="1" lower="-2.62" upper="2.62" />
+            <limit effort="1" velocity="1" lower="-2.62" upper="2.62" />
             <dynamics damping="50" friction="1"/>
         </joint>
@@ -250,5 +250,5 @@
             <origin xyz="0.0 0.0 ${link3_len}" rpy="0 0 0" />
             <axis xyz="1 0 0" />
-            <limit effort="30" velocity="1" lower="-2.62" upper="2.62" />
+            <limit effort="1" velocity="1" lower="-2.62" upper="2.62" />
             <dynamics damping="50" friction="1"/>
         </joint>
@@ -276,5 +276,5 @@
             <origin xyz="0.0 0.0 ${link4_len}" rpy="0 0 0" />
             <axis xyz="1 0 0" />
-            <limit effort="30" velocity="1" lower="-2.62" upper="2.62" />
+            <limit effort="1" velocity="1" lower="-2.62" upper="2.62" />
             <dynamics damping="50" friction="1"/>
         </joint>
@@ -302,5 +302,5 @@
             <origin xyz="0 0 ${link5_len}" rpy="0 0 0" />
             <axis xyz="0 0 1" />
-            <limit effort="30" velocity="1" lower="-6.28" upper="6.28" />
+            <limit effort="1" velocity="1" lower="-6.28" upper="6.28" />
             <dynamics damping="50" friction="1"/>
         </joint>
@@ -328,5 +328,5 @@
             <origin xyz="0 ${link6_width} ${link6_len}" rpy="0 0 0"/>
             <axis xyz="0 -1 0"/>
-            <limit lower="0" upper="0.04" effort="5" velocity="0.5"/>
+            <limit lower="0" upper="0.04" effort="1" velocity="0.5"/>
             <dynamics damping="50" friction="1"/>
         </joint>
@@ -336,5 +336,5 @@
             <origin xyz="0 -${link6_width} ${link6_len}" rpy="0 0 ${M_PI}"/>
             <axis xyz="0 -1 0"/>
-            <limit lower="0" upper="0.04" effort="5" velocity="0.5"/>
+            <limit lower="0" upper="0.04" effort="1" velocity="0.5"/>
             <dynamics damping="50" friction="1"/>
         </joint>
